File: hw/peelight.sch (EAGLE design)
At the start: 9 parts, among them U1 ATTINY85-20PU, U2 BATTERY-CHARGER-LI-PROT, U3 LED-8XRGB-LINE, U4 LED-8XRGB-LINE, U5 LED-8XRGB-LINE, U6 MOTION-PIR-DYP-ME003

Commit message: x
Parts:
- added C1: (no value), con-amp-mt:L02P
- added C2, C3: (no value), con-amp-mt:S02P
Connections:
- new net N$10: BT1.-, C2-1.S
- new net N$11: BT1.+, C2-2.S
- new net N$12: C3-2.S, U2.IN-
- new net N$13: C3-1.S, U2.IN+
- net N$1: now also C1-2.S; no longer BT1.+
- net N$2: now also C1-1.S; no longer BT1.-
Other:
- moved on the sheet: BT1
Changed lines of the file:
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@@
 <part name="U4" library="diy-modules" library_urn="urn:adsk.eagle:library:15904242" deviceset="LED-8XRGB-LINE" device="" package3d_urn="urn:adsk.eagle:package:15904530/1"/>
 <part name="R1" library="SparkFun-Resistors" library_urn="urn:adsk.eagle:library:532" deviceset="RESISTOR" device="AXIAL-0.3" package3d_urn="urn:adsk.eagle:package:39658/1" value=" "/>
+<part name="C1" library="con-amp-mt" library_urn="urn:adsk.eagle:library:123" deviceset="L02P" device="" package3d_urn="urn:adsk.eagle:package:5777/1"/>
+<part name="C2" library="con-amp-mt" library_urn="urn:adsk.eagle:library:123" deviceset="S02P" device="" package3d_urn="urn:adsk.eagle:package:5789/1"/>
+<part name="C3" library="con-amp-mt" library_urn="urn:adsk.eagle:library:123" deviceset="S02P" device="" package3d_urn="urn:adsk.eagle:package:5789/1"/>
 </parts>
 <sheets>
@@
 <attribute name="NAME" x="78.746340625" y="69.8595" size="2.542109375" layer="95" rot="MR0"/>
 </instance>
-<instance part="BT1" gate="G$1" x="48.26" y="58.42" smashed="yes" rot="R270">
-<attribute name="NAME" x="52.578" y="58.42" size="1.778" layer="95" font="vector" rot="R270" align="bottom-center"/>
-<attribute name="VALUE" x="43.942" y="58.42" size="1.778" layer="96" font="vector" rot="R270" align="top-center"/>
+<instance part="BT1" gate="G$1" x="45.72" y="-2.54" smashed="yes" rot="R180">
+<attribute name="NAME" x="45.72" y="-6.858" size="1.778" layer="95" font="vector" rot="R180" align="bottom-center"/>
+<attribute name="VALUE" x="45.72" y="1.778" size="1.778" layer="96" font="vector" rot="R180" align="top-center"/>
 </instance>
 <instance part="U6" gate="G$1" x="91.44" y="10.16" smashed="yes" rot="MR180">
@@
 <attribute name="NAME" x="100.076" y="53.34" size="1.778" layer="95" font="vector" rot="R90" align="bottom-center"/>
 <attribute name="VALUE" x="100.584" y="53.34" size="0.6096" layer="96" font="vector" rot="R90" align="top-center"/>
+</instance>
+<instance part="C1" gate="-1" x="40.64" y="25.4" smashed="yes" rot="R90">
+<attribute name="NAME" x="39.624" y="24.892" size="1.778" layer="95" rot="R270"/>
+<attribute name="VALUE" x="43.053" y="25.654" size="1.778" layer="96" rot="R90"/>
+</instance>
+<instance part="C1" gate="-2" x="50.8" y="25.4" smashed="yes" rot="R90">
+<attribute name="NAME" x="49.784" y="24.892" size="1.778" layer="95" rot="R270"/>
+<attribute name="VALUE" x="53.213" y="25.654" size="1.778" layer="96" rot="R90"/>
+</instance>
+<instance part="C2" gate="-1" x="40.64" y="10.16" smashed="yes" rot="R270">
+<attribute name="NAME" x="41.656" y="10.668" size="1.778" layer="95" rot="R90"/>
+<attribute name="VALUE" x="38.227" y="9.906" size="1.778" layer="96" rot="R270"/>
+</instance>
+<instance part="C2" gate="-2" x="50.8" y="10.16" smashed="yes" rot="R270">
+<attribute name="NAME" x="51.816" y="10.668" size="1.778" layer="95" rot="R90"/>
+<attribute name="VALUE" x="48.387" y="9.906" size="1.778" layer="96" rot="R270"/>
+</instance>
+<instance part="C3" gate="-1" x="-7.62" y="66.04" smashed="yes">
+<attribute name="NAME" x="-8.128" y="67.056" size="1.778" layer="95" rot="R180"/>
+<attribute name="VALUE" x="-7.366" y="63.627" size="1.778" layer="96"/>
+</instance>
+<instance part="C3" gate="-2" x="-7.62" y="50.8" smashed="yes">
+<attribute name="NAME" x="-8.128" y="51.816" size="1.778" layer="95" rot="R180"/>
+<attribute name="VALUE" x="-7.366" y="48.387" size="1.778" layer="96"/>
 </instance>
 </instances>
@@
 </busses>
 <nets>
-<net name="N$1" class="0">
-<segment>
-<pinref part="U2" gate="G$1" pin="B+"/>
-<wire x1="35.56" y1="60.96" x2="40.64" y2="60.96" width="0.1524" layer="91"/>
-<pinref part="BT1" gate="G$1" pin="+"/>
-<wire x1="40.64" y1="60.96" x2="40.64" y2="63.5" width="0.1524" layer="91"/>
-<wire x1="40.64" y1="63.5" x2="48.26" y2="63.5" width="0.1524" layer="91"/>
-</segment>
-</net>
-<net name="N$2" class="0">
-<segment>
-<pinref part="U2" gate="G$1" pin="B-"/>
-<wire x1="35.56" y1="55.88" x2="40.64" y2="55.88" width="0.1524" layer="91"/>
-<wire x1="40.64" y1="55.88" x2="40.64" y2="53.34" width="0.1524" layer="91"/>
-<pinref part="BT1" gate="G$1" pin="-"/>
-<wire x1="40.64" y1="53.34" x2="48.26" y2="53.34" width="0.1524" layer="91"/>
-</segment>
-</net>
 <net name="N$3" class="0">
 <segment>
@@
 </segment>
 </net>
+<net name="N$1" class="0">
+<segment>
+<pinref part="U2" gate="G$1" pin="B+"/>
+<wire x1="35.56" y1="60.96" x2="50.8" y2="60.96" width="0.1524" layer="91"/>
+<wire x1="50.8" y1="60.96" x2="50.8" y2="30.48" width="0.1524" layer="91"/>
+<pinref part="C1" gate="-2" pin="S"/>
+</segment>
+</net>
+<net name="N$2" class="0">
+<segment>
+<wire x1="40.64" y1="30.48" x2="40.64" y2="55.88" width="0.1524" layer="91"/>
+<pinref part="U2" gate="G$1" pin="B-"/>
+<wire x1="40.64" y1="55.88" x2="35.56" y2="55.88" width="0.1524" layer="91"/>
+<pinref part="C1" gate="-1" pin="S"/>
+</segment>
+</net>
+<net name="N$10" class="0">
+<segment>
+<pinref part="C2" gate="-1" pin="S"/>
+<pinref part="BT1" gate="G$1" pin="-"/>
+<wire x1="40.64" y1="-2.54" x2="40.64" y2="5.08" width="0.1524" layer="91"/>
+</segment>
+</net>
+<net name="N$11" class="0">
+<segment>
+<pinref part="BT1" gate="G$1" pin="+"/>
+<pinref part="C2" gate="-2" pin="S"/>
+<wire x1="50.8" y1="5.08" x2="50.8" y2="-2.54" width="0.1524" layer="91"/>
+</segment>
+</net>
+<net name="N$12" class="0">
+<segment>
+<pinref part="U2" gate="G$1" pin="IN-"/>
+<pinref part="C3" gate="-2" pin="S"/>
+<wire x1="-2.54" y1="50.8" x2="2.54" y2="50.8" width="0.1524" layer="91"/>
+</segment>
+</net>
+<net name="N$13" class="0">
+<segment>
+<pinref part="U2" gate="G$1" pin="IN+"/>
+<pinref part="C3" gate="-1" pin="S"/>
+<wire x1="-2.54" y1="66.04" x2="2.54" y2="66.04" width="0.1524" layer="91"/>
+</segment>
+</net>
